File: CANBus/CANBus.sch (KiCad schematic (older format))
At the start: 17 parts, among them J6 Screw_Terminal_1x03, J7 DB9_FEMALE, U7 MCP2515-E/ST, Y2 16Mhz

Commit message: added CreativeCommons License
Other:
- note added: "Released under the Creative Commons\nAttribution-ShareAlike 4.0 International (CC BY-SA 4.0) \nhttps://creativecommons.org/licenses/by-sa/4.0/"
Changed lines of the file:
@@
 LIBS:contrib
 LIBS:valves
+LIBS:graphic_symbols
 LIBS:CANBus-cache
 EELAYER 25 0
@@
 Wire Wire Line
 	8500 2400 8750 2400
-Text Notes 7100 6700 0    60   ~ 0
+Text Notes 7400 7500 0    60   ~ 0
 Canbus Transceiver compatible to Raspberry 3V
 Wire Wire Line
@@
 F 0 "JP1" V 8250 1600 50  0000 C CNN
 F 1 "JUMPER" V 8150 1550 50  0000 C CNN
-F 2 "Pin_Headers:Pin_Header_Straight_1x02" V 8050 950 50  0000 C CNN
+F 2 "Pin_Headers:Pin_Header_Straight_1x02" V 8050 950 50  0001 C CNN
 F 3 "" H 8200 1750 50  0000 C CNN
 	1    8200 1750
@@
 	1    0    0    -1
 $EndComp
+Text Notes 7100 7000 0    79   ~ 0
+Released under the Creative Commons\nAttribution-ShareAlike 4.0 International (CC BY-SA 4.0) \nhttps://creativecommons.org/licenses/by-sa/4.0/
+$Comp
+L Logo_Open_Hardware_Small #LOGO?
+U 1 1 59A1F946
+P 10900 6850
+F 0 "#LOGO?" H 10900 7125 50  0001 C CNN
+F 1 "open hardware" H 10900 6625 50  0000 C CNN
+F 2 "" H 10900 6850 50  0001 C CNN
+F 3 "" H 10900 6850 50  0001 C CNN
+	1    10900 6850
+	1    0    0    -1
+$EndComp
